Commit message: recolocar los stl

File: simulations/armpi_ultra_description/urdf/armpi_ultra.urdf (robot description, URDF)
Before this commit: robot 44 001, 14 links, 13 joints
Links:
- link base_link: geometry collision mesh filename=meshes/base_link.STL; visual mesh filename=meshes/base_link.STL
- link camera_connet_link: geometry collision mesh filename=meshes/camera_connet_link.STL; visual mesh filename=meshes/camera_connet_link.STL
- link gripper_link: geometry collision mesh filename=meshes/gripper_link.STL; visual mesh filename=meshes/gripper_link.STL
- link l_in_link: geometry collision mesh filename=meshes/l_in_link.STL; visual mesh filename=meshes/l_in_link.STL
- link l_link: geometry collision mesh filename=meshes/l_link.STL; visual mesh filename=meshes/l_link.STL
- link l_out_link: geometry collision mesh filename=meshes/l_out_link.STL; visual mesh filename=meshes/l_out_link.STL
- link link1: geometry collision mesh filename=meshes/link1.STL; visual mesh filename=meshes/link1.STL
- link link2: geometry collision mesh filename=meshes/link2.STL; visual mesh filename=meshes/link2.STL
- link link3: geometry collision mesh filename=meshes/link3.STL; visual mesh filename=meshes/link3.STL
- link link4: geometry collision mesh filename=meshes/link4.STL; visual mesh filename=meshes/link4.STL
- link link5: geometry collision mesh filename=meshes/link5.STL; visual mesh filename=meshes/link5.STL
- link r_in_link: geometry collision mesh filename=meshes/r_in_link.STL; visual mesh filename=meshes/r_in_link.STL
- link r_link: geometry collision mesh filename=meshes/r_link.STL; visual mesh filename=meshes/r_link.STL
- link r_out_link: geometry collision mesh filename=meshes/r_out_link.STL; visual mesh filename=meshes/r_out_link.STL
Joints:
- removed joint l_out_link
- added joint l_out_joint: type revolute, parent l_in_link, child l_out_link, origin xyz=0.00035154 0.016298 0.023984 rpy=0 0 0, axis 0.99992 -0.0087259 -0.0087265, limit lower=-1.57 upper=1.57 effort=1000 velocity=10
- joint joint1: axis 0 0 0 -> 0 0 1; type fixed -> revolute
