Commit message: Escena del gemelo digital y paquete MoveIt (estado antes de optimizar rendimiento)
- arm_moveit_config: paquete MoveIt 2 con entorno parametrico (mesa + persona)
  generado desde config/scene_params.yaml, launch de Gazebo con camara RGB-D.
- Maniqui con cara maniqui_mia.stl simplificado a 25k triangulos (escala 1.20,
  offset centrado sobre la colision del torso).
- Tenedor como efector final (tenedor_link.stl), sin pinza ni copias antiguas
  de URDF.
- aurora930: TF de la camara colgado de rgb_camera_link de la URDF.

Co-Authored-By: Claude Opus 5.5 <noreply@anthropic.com>

File: simulations/armpi_ultra_description/urdf/armpi_ultra.xacro (robot description, xacro)
@@ -168,63 +168,65 @@
     <limit effort="1000" lower="-2.09" upper="2.09" velocity="10"/>
   </joint>
-  <link
-    name="gripper_link">
-    <inertial>
-      <origin
-        xyz="0.0145481835889059 -0.00315257290321308 0.0253492053712461"
-        rpy="0 0 0" />
-      <mass
-        value="0.0174988490314194" />
-      <inertia
-        ixx="4.12615692688456E-06"
-        ixy="-2.75102939068049E-08"
-        ixz="-7.61180742281118E-09"
-        iyy="1.57023365316943E-06"
-        iyz="2.2563082379695E-08"
-        izz="3.2612101868791E-06" />
-    </inertial>
-    <visual>
-      <origin
-        xyz="0 0 0"
-        rpy="0 0 0" />
-      <geometry>
-        <mesh
-          filename="file://$(find armpi_ultra_description)/meshes/gripper_link.STL" />
-      </geometry>
-        <material name="">
-            <color rgba="0.792156862745098 0.819607843137255 0.933333333333333 1"/>
-      </material>
-    </visual>
-    <collision>
-      <origin
-        xyz="0 0 0"
-        rpy="0 0 0" />
-      <geometry>
-        <mesh
-          filename="file://$(find armpi_ultra_description)/meshes/gripper_link_collision.stl" />
-      </geometry>
-    </collision>
-  </link>
-  <joint
-    name="gripper_joint"
-    type="fixed">
-    <origin
-      xyz="0 0 0.0054388"
-      rpy="0 0 0" />
-    <parent
-      link="link5" />
-    <child
-      link="gripper_link" />
-    <axis
-      xyz="0 0 0" />
-  </joint>
-  <!-- end effector link -->
+  <!-- end_effector_link: punto funcional (TCP) que usa MoveIt para la bola
+       interactiva y el "tip_link" del grupo "arm" en la SRDF. Es un frame
+       puro (sin malla ni colisión) para no confundirlo ni con link5 (el
+       último motor) ni con la punta absoluta de la malla del tenedor.
+       El padre sigue siendo link5 (no se toca la cinemática del robot);
+       el offset es a lo largo de Z local, el mismo eje longitudinal por
+       el que se monta tenedor_link con offset 0 (ver más abajo), así que
+       este valor se mide igual desde la base del tenedor.
+       Longitud total del tenedor (base en link5 -> punta de los dientes):
+       0.15 m. Punto funcional deseado: línea media de los dientes, un
+       poco retrasado respecto a la punta para que el planificador no
+       intente colisionar justo el borde extremo -> 13.5/15 de la
+       longitud = 0.135 m, dejando 0.015 m (1.5 cm) de margen hasta la
+       punta física real. -->
   <link name="end_effector_link" />
   <joint name="end_effector_joint" type="fixed">
-    <origin xyz="0 0 0.08" rpy="0 0 0"/>
+    <origin xyz="0.02 0 0.135" rpy="0 0 0"/>
     <parent link="link5"/>
     <child link="end_effector_link"/>
   </joint>
-  <link name="camera_connet_link">
+  <!-- Tenedor: herramienta terminal para asistencia en alimentación.
+       Montado directamente sobre link5, offset 0 porque la malla de link5
+       apenas sobresale (~0.17 mm) por encima de su propio origen; casi todo
+       su volumen queda por debajo, así que offset 0 es lo que deja el tenedor
+       pegado a la cara superior real de link5, sin hueco visible.
+       (Antes se usó 0.0054388 m, tomado de un fichero de referencia pensado
+       para el gripper mecánico antiguo, pero dejaba ~5 mm de hueco flotando.)
+       El STL visual está exportado en milímetros, de ahí el scale 0.001; el resto
+       de mallas de este fichero ya vienen en metros. La colisión usa la misma
+       malla que el visual (antes se reutilizaba gripper_link_collision.stl, un
+       casquillo de solo ~5.5 cm pensado para el gripper mecánico antiguo, que
+       dejaba sin proteger la mitad de la pala del tenedor de ~15 cm).
+       Masa/inercia: valor estimado, no hay datos CAD reales de esta pieza. -->
+  <link name="tenedor_link">
+    <inertial>
+      <origin rpy="0 0 0" xyz="0 0 0.06"/>
+      <mass value="0.01"/>
+      <inertia ixx="1e-6" ixy="0" ixz="0" iyy="1e-6" iyz="0" izz="1e-6"/>
+    </inertial>
+    <visual>
+      <origin rpy="0 0 0" xyz="0 0 0"/>
+      <geometry>
+        <mesh filename="file://$(find armpi_ultra_description)/meshes/tenedor_link.stl" scale="0.001 0.001 0.001"/>
+      </geometry>
+      <material name="">
+        <color rgba="0.792156862745098 0.819607843137255 0.933333333333333 1"/>
+      </material>
+    </visual>
+    <collision>
+      <origin rpy="0 0 0" xyz="0 0 0"/>
+      <geometry>
+        <mesh filename="file://$(find armpi_ultra_description)/meshes/tenedor_link.stl" scale="0.001 0.001 0.001"/>
+      </geometry>
+    </collision>
+  </link>
+  <joint name="tenedor_joint" type="fixed">
+    <origin xyz="0 0 0" rpy="0 0 0"/>
+    <parent link="link5"/>
+    <child link="tenedor_link"/>
+  </joint>
+  <link name="rgb_camera_link">
     <inertial>
       <origin rpy="0 0 0" xyz="0.0118021523166905 -0.000540782293006269 0.00995705328357074"/>
@@ -244,4 +246,7 @@
       <origin rpy="0 0 0" xyz="0 0 0"/>
       <geometry>
+        <!-- Antes apuntaba a aurora_camera_joint.STL, que no existe (salia
+             "Error retrieving file" al lanzar y la camara se quedaba sin
+             colision). Se usa la misma malla que el visual. -->
         <mesh filename="file://$(find armpi_ultra_description)/meshes/camera_connet_link.STL"/>
       </geometry>
@@ -251,7 +256,66 @@
     <origin rpy="0 -1.5614 0" xyz="-0.040352 -0.019122 0.048005"/>
     <parent link="link4"/>
-    <child link="camera_connet_link"/>
-    <axis xyz="0 0 0"/>
-  </joint>
-  <xacro:include filename="$(find armpi_ultra_description)/urdf/gripper.urdf.xacro"/>
+    <child link="rgb_camera_link"/>
+  </joint>
+  <!-- ============== CAMARA: frames de la lente + sensor simulado ==============
+       rgb_camera_link es la pieza fisica de la camara Aurora930
+       (camera_connet_link.STL), atornillada a link4 (el ultimo motor, ver
+       meshes/README_MESHES.md), asi que se mueve con el brazo.
+       En su malla la cara de las lentes esta en x = +0.0227 m y mira hacia +X
+       (= eje longitudinal de link4, la misma direccion que el tenedor); las
+       lentes estan centradas en y = 0, z = +0.010 m.
+       camara_link: centro de la lente, convenio ROS (X adelante, Z arriba).
+       camara_optical_frame: mismo punto, convenio de imagen (Z adelante,
+       X derecha, Y abajo); es el frame_id de las imagenes simuladas.
+       Nombres propios (no depth_cam_*_optical_frame) a proposito: el driver
+       real de la camara (peripherals/launch/include/aurora930.launch.py)
+       ya publica esos frames por TF estatico desde rgb_camera_link y, si el
+       URDF los repitiera, chocarian dos padres en el arbol TF con el robot
+       real. -->
+  <link name="camara_link"/>
+  <joint name="camara_joint" type="fixed">
+    <origin rpy="0 0 0" xyz="0.0227 0 0.010"/>
+    <parent link="rgb_camera_link"/>
+    <child link="camara_link"/>
+  </joint>
+  <link name="camara_optical_frame"/>
+  <joint name="camara_optical_joint" type="fixed">
+    <origin rpy="${-pi/2} 0 ${-pi/2}" xyz="0 0 0"/>
+    <parent link="camara_link"/>
+    <child link="camara_optical_frame"/>
+  </joint>
+  <!-- Sensor de camara RGB-D para Gazebo Fortress (ignition-gazebo 6, el que
+       corresponde a ROS 2 Humble; Gazebo Classic esta descontinuado). MoveIt
+       y RViz ignoran este bloque; solo lo usa Gazebo
+       (arm_moveit_config/launch/gazebo.launch.py). Gazebo publica en sus
+       propios topics (camara/image, camara/depth_image, camara/points,
+       camara/camera_info) y ese launch los pasa a ROS (ros_gz_bridge) con los
+       MISMOS nombres que la camara real, para que el codigo de percepcion
+       funcione igual en simulacion y con el robot:
+         /depth_cam/rgb/image_raw, /depth_cam/rgb/camera_info,
+         /depth_cam/depth/image_raw, /depth_cam/depth_registered/points
+       Resolucion/FOV aproximados de la Aurora930 (640x480, ~70 grados).
+       Las articulaciones (y por tanto /joint_states y el TF de la camara) las
+       gestiona gz_ros2_control, ver config/armpi_ultra.urdf.xacro. -->
+  <gazebo reference="camara_link">
+    <sensor name="camara_rgbd" type="rgbd_camera">
+      <always_on>true</always_on>
+      <update_rate>15</update_rate>
+      <visualize>false</visualize>
+      <topic>camara</topic>
+      <ignition_frame_id>camara_optical_frame</ignition_frame_id>
+      <camera>
+        <horizontal_fov>1.2217</horizontal_fov>
+        <image>
+          <width>640</width>
+          <height>480</height>
+          <format>R8G8B8</format>
+        </image>
+        <clip>
+          <near>0.05</near>
+          <far>5.0</far>
+        </clip>
+      </camera>
+    </sensor>
+  </gazebo>
 </robot>
